File: breadbat.kicad_sch (KiCad schematic)
At the start: 31 parts, among them J1 USB_C_Receptacle_PowerOnly_6P, J2 Conn_02x03_Odd_Even, J3 Conn_02x03_Odd_Even, U1 TP4056-42-ESOP8, U2 AMS1117-3.3, U3 TPS259621

Commit message: Added README
Added readme and added a BOM
Parts:
- BT1: LCSC / JLC Part (none) -> C131337; Manufacturer (none) -> JST; Part Number (none) -> B2B-PH-K-S(LF)(SN)
- C1, C2: LCSC / JLC Part (none) -> C19702; Manufacturer (none) -> Samsung; Part Number (none) -> CL10A106KP8NNNC
- C3: value 100n -> 1u; LCSC / JLC Part (none) -> C15849; Manufacturer (none) -> Samsung; Part Number (none) -> CL10A105KB8NNNC
- C4, C5: LCSC / JLC Part (none) -> C45783; Manufacturer (none) -> Samsung; Part Number (none) -> CL21A226MAQNNNE
- C6: LCSC / JLC Part (none) -> C15849; Manufacturer (none) -> Samsung; Part Number (none) -> CL10A105KB8NNNC
- D2: LCSC / JLC Part (none) -> C2287; Manufacturer (none) -> Kento; Part Number (none) -> KT-0603Y
- D4: LCSC / JLC Part (none) -> C2290; Manufacturer (none) -> Kento; Part Number (none) -> KT-0603W
- D5: LCSC / JLC Part (none) -> C2286; Manufacturer (none) -> Kento; Part Number (none) -> KT-0603R
- J1: LCSC / JLC Part (none) -> C2927302; Manufacturer (none) -> YIYUAN; Part Number (none) -> YTC-TC6S-231
- J2, J3: LCSC / JLC Part (none) -> C492420; Manufacturer (none) -> XFCN; Part Number (none) -> PZ254V-12-6P
- R1, R11, R4, R7: LCSC / JLC Part (none) -> C22765; Manufacturer (none) -> UNI-ROYAL; Part Number (none) -> 0603WAF1201T5E
- R10, R8: LCSC / JLC Part (none) -> C25819; Manufacturer (none) -> UNI-ROYAL; Part Number (none) -> 0603WAF4702T5E
- R2, R3: LCSC / JLC Part (none) -> C23186; Manufacturer (none) -> UNI-ROYAL; Part Number (none) -> 0603WAF5101T5E
- R5: LCSC / JLC Part (none) -> C23231; Manufacturer (none) -> UNI-ROYAL; Part Number (none) -> 0603WAF6802T5E
- R6: LCSC / JLC Part (none) -> C25808; Manufacturer (none) -> UNI-ROYAL; Part Number (none) -> 0603WAF1203T5E
- R9: LCSC / JLC Part (none) -> C22978; Manufacturer (none) -> UNI-ROYAL; Part Number (none) -> 0603WAF3301T5E
- U1: LCSC / JLC Part (none) -> C16581; Manufacturer (none) -> TOPPOWER; Part Number (none) -> TP4056-42-ESOP8
- U2: LCSC / JLC Part (none) -> C347222; Manufacturer (none) -> UMW; Part Number (none) -> AMS1117-3.3
- U3: LCSC / JLC Part (none) -> C2155774; Manufacturer (none) -> Texas Instruments; Part Number (none) -> TPS259621DDAR
